Commit message: Add files via upload

File: spider/urdf/originals/spider.urdf (robot description, URDF)
Before this commit: robot spider, 13 links, 12 joints
Links:
- link b11: mass 0.0073206 -> 0.00732061922605988
- link b22: mass 0.0073206 -> 0.00732061922605988
- link b222: mass 0.013124 -> 0.0131238914966797
- link base_link: mass 0.065616 -> 0.0656164141863128
- link f1: mass 0.011831 -> 0.0118311157008267
- link f222: mass 0.013124 -> 0.0131238943756469
Joints:
- joint b111_joint: limit lower=-3.14 upper=3.14 effort=5 velocity=1 -> lower=-3.14 upper=3.14 effort=0 velocity=0
- joint b11_joint: limit lower=-3.14 upper=3.14 effort=5 velocity=1 -> lower=-3.14 upper=3.14 effort=0 velocity=0
- joint b1_joint: limit lower=-3.14 upper=3.14 effort=5 velocity=1 -> lower=-3.14 upper=3.14 effort=0 velocity=0
- joint b222_joint: limit lower=-3.14 upper=3.14 effort=5 velocity=1 -> lower=-3.14 upper=3.14 effort=0 velocity=0
- joint b22_joint: limit lower=-3.14 upper=3.14 effort=5 velocity=1 -> lower=-3.14 upper=3.14 effort=0 velocity=0
- joint b2_joint: limit lower=-3.14 upper=3.14 effort=5 velocity=1 -> lower=-3.14 upper=3.14 effort=0 velocity=0
- joint f111_joint: limit lower=-3.14 upper=3.14 effort=5 velocity=1 -> lower=-3.14 upper=3.14 effort=0 velocity=0
- joint f11_joint: limit lower=-3.14 upper=3.14 effort=5 velocity=1 -> lower=-3.14 upper=3.14 effort=0 velocity=0
- joint f1_joint: limit lower=-3.14 upper=3.14 effort=5 velocity=1 -> lower=-3.14 upper=3.14 effort=0 velocity=0
- joint f222_joint: limit lower=-3.14 upper=3.14 effort=5 velocity=1 -> lower=-3.14 upper=3.14 effort=0 velocity=0
- joint f22_joint: limit lower=-3.14 upper=3.14 effort=5 velocity=1 -> lower=-3.14 upper=3.14 effort=0 velocity=0
- joint f2_joint: limit lower=-3.14 upper=3.14 effort=5 velocity=1 -> lower=-3.14 upper=3.14 effort=0 velocity=0

File: spider/urdf/spider1.urdf (robot description, URDF)
Before this commit: robot spider, 13 links, 12 joints
Links:
- link b1: geometry collision mesh filename=package://spider/meshes/b1.STL; visual mesh filename=package://spider/meshes/b1.STL
- link b11: geometry collision mesh filename=package://spider/meshes/b11.STL; visual mesh filename=package://spider/meshes/b11.STL
- link b111: geometry collision mesh filename=package://spider/meshes/b111.STL; visual mesh filename=package://spider/meshes/b111.STL
- link b2: mass 0.0118311153256473 -> 0; geometry collision mesh filename=package://spider/meshes/b2.STL; visual mesh filename=package://spider/meshes/b2.STL
- link b22: geometry collision mesh filename=package://spider/meshes/b22.STL; visual mesh filename=package://spider/meshes/b22.STL
- link b222: geometry collision mesh filename=package://spider/meshes/b222.STL; visual mesh filename=package://spider/meshes/b222.STL
- link base_link: geometry collision mesh filename=package://spider/meshes/base_link.STL; visual mesh filename=package://spider/meshes/base_link.STL
- link f1: geometry collision mesh filename=package://spider/meshes/f1.STL; visual mesh filename=package://spider/meshes/f1.STL
- link f11: geometry collision mesh filename=package://spider/meshes/f11.STL; visual mesh filename=package://spider/meshes/f11.STL
- link f111: geometry collision mesh filename=package://spider/meshes/f111.STL; visual mesh filename=package://spider/meshes/f111.STL
- link f2: geometry collision mesh filename=package://spider/meshes/f2.STL; visual mesh filename=package://spider/meshes/f2.STL
- link f22: geometry collision mesh filename=package://spider/meshes/f22.STL; visual mesh filename=package://spider/meshes/f22.STL
- link f222: geometry collision mesh filename=package://spider/meshes/f222.STL; visual mesh filename=package://spider/meshes/f222.STL
Joints:
- joint b111_joint: limit lower=-3.14 upper=3.14 effort=5 velocity=1 -> lower=-3.14 upper=3.14 effort=1 velocity=1
- joint b11_joint: limit lower=-3.14 upper=3.14 effort=5 velocity=1 -> lower=-3.14 upper=3.14 effort=1 velocity=1
- joint b1_joint: limit lower=-3.14 upper=3.14 effort=5 velocity=1 -> lower=-3.14 upper=3.14 effort=1 velocity=1
- joint b222_joint: limit lower=-3.14 upper=3.14 effort=5 velocity=1 -> lower=-3.14 upper=3.14 effort=1 velocity=1
- joint b22_joint: limit lower=-3.14 upper=3.14 effort=5 velocity=1 -> lower=-3.14 upper=3.14 effort=1 velocity=1
- joint b2_joint: limit lower=-3.14 upper=3.14 effort=5 velocity=1 -> lower=-3.14 upper=3.14 effort=1 velocity=1
- joint f111_joint: limit lower=-3.14 upper=3.14 effort=5 velocity=1 -> lower=-3.14 upper=3.14 effort=1 velocity=1
- joint f11_joint: limit lower=-3.14 upper=3.14 effort=5 velocity=1 -> lower=-3.14 upper=3.14 effort=1 velocity=1
- joint f1_joint: limit lower=-3.14 upper=3.14 effort=5 velocity=1 -> lower=-3.14 upper=3.14 effort=1 velocity=1
- joint f222_joint: limit lower=-3.14 upper=3.14 effort=5 velocity=1 -> lower=-3.14 upper=3.14 effort=1 velocity=1
- joint f22_joint: limit lower=-3.14 upper=3.14 effort=5 velocity=1 -> lower=-3.14 upper=3.14 effort=1 velocity=1
- joint f2_joint: limit lower=-3.14 upper=3.14 effort=5 velocity=1 -> lower=-3.14 upper=3.14 effort=1 velocity=1
